File: schematic/adc_io.kicad_sch (KiCad schematic)
At the start: 20 parts, among them U6 NJM2114, U7 NJM2114

Commit message: Redesign schematic to 3ch: DRV8825x3, AM26LV32 differential encoder, swap ADC3/ADC4
- DRV8825 stepper driver: 4ch -> 3ch (STEP/DIR CH0-2 on GPIO6-11)
- Encoder: 3ch differential input via AM26LV32IDR for Stepperonline 17HS15-1504-ME1K (1000PPR)
  - A+/A-, B+/B-, Z+/Z- differential pairs, GPIO15-17/18/21/35/36-37/40
- ADC assignment swap: GPIO4=MOT_V(ADC3) voltage monitor, GPIO5=CURRENT(ADC4) 100mOhm+20x amp
- Updated Gerber files (Gerber202960613 replaces Gerber202960504)
- Added AM26LV32IDR and AM26C32INSR library files
- Updated REQUIREMENTS.md: 3ch axis range, encoder specs, ADC channel table, current conversion formula
- Updated CLAUDE.md: corrected GPIO4/5 signal assignments and startup sequence

Co-Authored-By: Claude Sonnet 4.6 <noreply@anthropic.com>
Parts:
- added C21, C22, C23, C24: 0.01u, Capacitor_SMD:C_0402_1005Metric, symbol Device:C_Small
- added C25: 0.1uF, Capacitor_SMD:C_0402_1005Metric, symbol Device:C_Small
- added R25, R26, R27, R28: 16k, Resistor_SMD:R_0402_1005Metric, symbol Device:R_Small
- added U8: NJM8532M, Package_SO:SOP-8_3.76x4.96mm_P1.27mm, symbol Amplifier_Operational:NJM2114
- U6, U7: value NJM2114 -> NJM8532M
Connections:
- net +3V3: now also C25.1, U8.8 (V+)
- net GND: now also C21.2, C22.2, C25.2, U8.4 (V-)
- new net: C22.1, R28.2, U8.3 (+)
- new net: C23.1, R25.2, R27.1
- new net: C21.1, R27.2, U8.5 (+)
- new net: C24.1, R26.2, R28.1
- new net ADC_4: C24.2, U8.1, U8.2 (-)
- new net ADC_5: C23.2, U8.6 (-), U8.7
- new net AIN_4: R26.1
- new net AIN_5: R25.1
