File: schematic/drivers.kicad_sch (KiCad schematic)
At the start: 12 parts, among them J30 MOTOR_CH0, J31 MOTOR_CH1, J32 MOTOR_CH2, J33 MOTOR_CH3

Commit message: Redesign schematic to 3ch: DRV8825x3, AM26LV32 differential encoder, swap ADC3/ADC4
- DRV8825 stepper driver: 4ch -> 3ch (STEP/DIR CH0-2 on GPIO6-11)
- Encoder: 3ch differential input via AM26LV32IDR for Stepperonline 17HS15-1504-ME1K (1000PPR)
  - A+/A-, B+/B-, Z+/Z- differential pairs, GPIO15-17/18/21/35/36-37/40
- ADC assignment swap: GPIO4=MOT_V(ADC3) voltage monitor, GPIO5=CURRENT(ADC4) 100mOhm+20x amp
- Updated Gerber files (Gerber202960613 replaces Gerber202960504)
- Added AM26LV32IDR and AM26C32INSR library files
- Updated REQUIREMENTS.md: 3ch axis range, encoder specs, ADC channel table, current conversion formula
- Updated CLAUDE.md: corrected GPIO4/5 signal assignments and startup sequence

Co-Authored-By: Claude Sonnet 4.6 <noreply@anthropic.com>
Parts:
- removed A4: DRV8825_CH3, Library:DRV8825_Driver, symbol SteppingMotorDriver_symbols:DRV8825_STEPSTICK
- removed C33: 100uF, Capacitor_THT:CP_Radial_D8.0mm_P3.50mm, symbol Device:C
- removed J33: MOTOR_CH3, Connector_JST:JST_XH_B4B-XH-A_1x04_P2.50mm_Vertical, symbol SteppingMotorDriver_symbols:MOTOR_CONN_1X4
- J30, J31, J32: footprint Connector_JST:JST_XH_B4B-XH-A_1x04_P2.50mm_Vertical -> Connector_JST:JST_XH_S4B-XH-A-1_1x04_P2.50mm_Horizontal
