File: schematic/mcu_usb.kicad_sch (KiCad schematic)
At the start: 31 parts, among them J1 5077CR-16SMC2-BK-TR, J5 Conn_01x04_Pin, J6 Conn_01x04_Pin, J7 Conn_01x04_Pin, J8 Conn_01x04_Pin, SW1 SW_Push, SW2 SW_Push, U1 NCP361SN, U2 ESP32-S3-WROOM-1, U3 MIC5219-3.3YM5

Commit message: Add firmware skeleton and update schematic: DIP switch removed, MS lines GPIO-driven
- MS0/MS1/MS2 now driven by ESP32-S3 GPIO (GPIO22/23/24) with 100Ω series resistors
- Remove DIP switch from schematic plan and PCB
- Add firmware scaffold: main, motor_ctrl, comm, config modules with sdkconfig
- Add CLAUDE.md project instructions and .gitignore
- Remove stale DRC/session files (SteppingMotorDriver.rules, .ses)

Co-Authored-By: Claude Sonnet 4.6 <noreply@anthropic.com>
Parts:
- added D1: LED, LED_SMD:LED_0603_1608Metric, symbol Device:LED
- added D2: RED LED, LED_SMD:LED_0603_1608Metric, symbol Device:LED
- added D3: YELLOW LED, LED_SMD:LED_0603_1608Metric, symbol Device:LED
- added R10, R11, R9: 1k, Resistor_SMD:R_0603_1608Metric, symbol Device:R_Small
Connections:
- net +3V3: now also R9.1
- net GND: now also D1.1 (K), D2.1 (K), D3.1 (K)
- net LED_RED: now reaches U2.16 (IO46)
- net LED_RED: now also R10.1
- net LED_YELLOW: now reaches U2.24 (IO47)
- net LED_YELLOW: now also R11.1
- new net: D1.2 (A), R9.2
- new net: D3.2 (A), R11.2
- new net: D2.2 (A), R10.2
- no-connect marks 9 -> 7

Commit message: Redesign schematic to 3ch: DRV8825x3, AM26LV32 differential encoder, swap ADC3/ADC4
- DRV8825 stepper driver: 4ch -> 3ch (STEP/DIR CH0-2 on GPIO6-11)
- Encoder: 3ch differential input via AM26LV32IDR for Stepperonline 17HS15-1504-ME1K (1000PPR)
  - A+/A-, B+/B-, Z+/Z- differential pairs, GPIO15-17/18/21/35/36-37/40
- ADC assignment swap: GPIO4=MOT_V(ADC3) voltage monitor, GPIO5=CURRENT(ADC4) 100mOhm+20x amp
- Updated Gerber files (Gerber202960613 replaces Gerber202960504)
- Added AM26LV32IDR and AM26C32INSR library files
- Updated REQUIREMENTS.md: 3ch axis range, encoder specs, ADC channel table, current conversion formula
- Updated CLAUDE.md: corrected GPIO4/5 signal assignments and startup sequence

Co-Authored-By: Claude Sonnet 4.6 <noreply@anthropic.com>
Parts:
- removed J8: Conn_01x04_Pin, Connector_JST:JST_PH_B4B-PH-K_1x04_P2.00mm_Vertical, symbol Connector:Conn_01x04_Pin
- added C26: 1uF, Capacitor_SMD:C_0603_1608Metric, symbol Device:C_Small
- added C27: 0.1uF, Capacitor_SMD:C_0603_1608Metric, symbol Device:C_Small
- added D7: CHU20S30, Diode_SMD:D_SOD-323_HandSoldering, symbol Device:D_Small
- added J8: Conn_01x02, Connector_JST:JST_PH_B2B-PH-K_1x02_P2.00mm_Vertical, symbol Connector_Generic:Conn_01x02
- added Q2: DMG3415, Package_TO_SOT_SMD:SOT-23, symbol Device:Q_PMOS_GSD
- added R23: 100k, Resistor_SMD:R_0603_1608Metric, symbol Device:R_Small
- R6, R8: footprint Inductor_SMD:L_0402_1005Metric -> Resistor_SMD:R_0603_1608Metric
- SW1: value SW_Push -> RESET
Connections:
- net DIR3 is gone; now on net DIR2: U2.19 (IO11)
- net ENC3_A is gone; now on net ENC2_A: U2.29 (IO36)
- net ENC3_B is gone; now on net ENC2_B: U2.30 (IO37)
- net STEP3 is gone; now on net STEP2: U2.18 (IO10)
- net ADC3: now also U2.4 (IO4); no longer U2.33 (IO40)
- net DIR0: now also U2.7 (IO7); no longer U2.5 (IO5)
- net DIR1: now also U2.17 (IO9); no longer U2.7 (IO7)
- net DIR2: no longer U2.17 (IO9)
- net ENC1_A: now also U2.11 (IO18); no longer U2.10 (IO17)
- net ENC1_B: now also U2.23 (IO21); no longer U2.11 (IO18)
- net ENC2_A: no longer U2.23 (IO21)
- net ENC2_B: no longer U2.28 (IO35)
- net GND: now also C26.2, C27.2, J8.2 (Pin_2), R23.1
- net STEP0: now also U2.6 (IO6); no longer U2.4 (IO4)
- net STEP1: now also U2.12 (IO8); no longer U2.6 (IO6)
- net STEP2: no longer U2.12 (IO8)
- net USB_5V: now also D7.2 (A), Q2.1 (G), R23.2; no longer U3.1 (IN), U3.3 (EN)
- new net: C26.1, C27.1, D7.1 (K), Q2.2 (S), U3.1 (IN), U3.3 (EN)
- new net 5V_IN: J8.1 (Pin_1), Q2.3 (D)
- new net ADC4: U2.5 (IO5)
- new net ENC0_Z: U2.10 (IO17)
- new net ENC1_Z: U2.28 (IO35)
- new net ENC2_Z: U2.33 (IO40)
Other:
- moved on the sheet: C2, C3, J1, R1, R2, R3, R4, U3
