File: schematic/mcu_usb.kicad_sch (KiCad schematic)
At the start: 42 parts, among them J1 5077CR-16SMC2-BK-TR, J5 Conn_01x04_Pin, J6 Conn_01x04_Pin, J7 Conn_01x04_Pin, J8 Conn_01x02, Q2 DMG3415, SW1 RESET, SW2 SW_Push, U1 NCP361SN, U2 ESP32-S3-WROOM-1, U3 MIC5219-3.3YM5

Commit message: Add status LED support, Multiplexer schematic, and Gerber export
Adds status_led.c/h for GPIO46/47 LED indicators, a Multiplexer
schematic sheet, exported Gerber fabrication files, and BLE Codex
prompt docs. Removes stale KiCad auto-backup zips.
Parts:
- removed J5, J6, J7: Conn_01x04_Pin, Connector_JST:JST_PH_B4B-PH-K_1x04_P2.00mm_Vertical, symbol Connector:Conn_01x04_Pin
- removed U3: MIC5219-3.3YM5, Package_TO_SOT_SMD:SOT-23-5, symbol Regulator_Linear:MIC5219-3.3YM5
- added C28, C29: 100uf, Capacitor_THT:CP_Radial_D5.0mm_P2.00mm, symbol Device:C_Polarized_Small
- added D9: SLEEP LED, LED_SMD:LED_0603_1608Metric, symbol Device:LED
- added R34: 1k, Resistor_SMD:R_0603_1608Metric, symbol Device:R_Small
- added U9: AMS1117-3.3, Package_TO_SOT_SMD:SOT-223-3_TabPin2, symbol Regulator_Linear:AMS1117-3.3
Connections:
- net +3V3: now also C28.1, U9.2 (VO)
- net DRV_SLEEP: now also R34.1
- net GND: now also C28.2, C29.2, D9.1 (K), U9.1 (GND)
- net at C26.1, C27.1, D7.1 (K)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: now also C29.1, U9.3 (VI)
- net I2C_MUL_RESET: now reaches U2.25 (IO48)
- new net: D9.2 (A), R34.2
- no-connect marks 7 -> 6
